File: vehicle/mkiii/hardware/lv/BSPD.kicad_sch (KiCad schematic)
At the start: 33 parts, among them K1 K_10A_5V, Q1 SSM3K333R,LF, Q2 SSM3K333R,LF, SW1 SW_Push_SPST_NO, SW2 SW_Push_SPST_NO, U2 SN74LVC1G08DBVR, U3 MCP6001T-I/LT, U4 SN74LVC1G02DBVR, U5 SN74LVC1G02DBVR

Commit message: Updated title blocks in schematic sheets to include author, set sheet titles, and merged throttle and brake shutdown sense sheets into a single sheet - Shutdown_Sensors.kicad_sch.
Other:
- title: (none) -> Brake System Plausibility Device (BSPD)
Changed lines of the file:
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@@
 	(generator_version "9.0")
 	(paper "A4")
+	(title_block
+		(title "Brake System Plausibility Device (BSPD)")
+		(comment 1 "By Leo Liao")
+	)
 	(text "Low pass filter,\nprevents jitter"
 		(exclude_from_sim no)
