File: vehicle/mkiii/hardware/lv/BrakeLight.kicad_sch (KiCad schematic)
At the start: 24 parts, among them Q3 SSM3K333R,LF, U6 MCP6001T-I/LT, U7 MCP6001T-I/LT, U8 MCP6001T-I/LT, U9 U_GATE_SN74LVC1G32DBVR

Commit message: Updated title blocks in schematic sheets to include author, set sheet titles, and merged throttle and brake shutdown sense sheets into a single sheet - Shutdown_Sensors.kicad_sch.
Other:
- title: (none) -> BrakeLight
Changed lines of the file:
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@@
 	(generator_version "9.0")
 	(paper "A4")
+	(title_block
+		(title "BrakeLight")
+		(comment 1 "By Leo Liao")
+	)
 	(text "		    VCC * R3\n    V_out = --------\n		    (R3 + R2)\n\n\n3.3 * 1kΩ / (10kΩ + 1kΩ) = 0.27V\n\nR_1 = 10kΩ; R_2 = 1kΩ"
 		(exclude_from_sim no)

Commit message: Small tweaks, refer to DOC.pdf provided by Henry Tejada Deras on 01/25/2026
Parts:
- removed C17: C_0.1uF, OEM:C_0603_1608Metric, symbol OEM:C_0.1uF_16V_0603
- removed R20: R_10k, OEM:R_0603_1608Metric, symbol OEM:R_10k_0.1W_0603
- removed U6: MCP6001T-I/LT, OEM:SOT-353_SC-70-5, symbol OEM:U_OpAmp_MCP6001T-ILT_SOT-353
Connections:
- net BRAKE_PRESS_SENSE: now also R21.1
- no-connect marks 1 -> 0
Other:
- note added: "VCC * R23 V_out = -------- (R22 + R23) 3.3 * 100Ω / (576Ω + 100Ω) = 0.488V R22 = 576Ω; R23 = 100Ω"
- note added: "VCC * R25 V_out = -------- (R24 + R25) 3.3 * 1kΩ / (10kΩ + 1kΩ) = 0.3V R24 = 10kΩ; R25 = 1kΩ"
- note removed: "Allows brake signal to remain accurate past RC lowpass filter."
- note removed: "Brakelight ON if pressure sensor is disconnected (pulled to 5V)"
- note removed: "Buffer"
- note removed: "VCC * R2 V_out = -------- (R1 + R2) 3.3 * 100Ω / (576Ω + 100Ω) = 0.488V R_1 = 576Ω; R_2 = 100Ω"
- note removed: "VCC * R3 V_out = -------- (R3 + R2) 3.3 * 1kΩ / (10kΩ + 1kΩ) = 0.27V R_1 = 10kΩ; R_2 = 1kΩ"
- moved on the sheet: C18, C19, C20, C21, C22, C23, Q3, R21, R22, R23, R24, R25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
