File: vehicle/mkiii/hardware/lv/microcontroller.kicad_sch (KiCad schematic)
At the start: 35 parts, among them J1 J_Programming_Pin_Header, U1 STM32G441CBT6, U12 MCP2561-E_SN, Y1 X_16MHz_18pF

Commit message: Updated title blocks in schematic sheets to include author, set sheet titles, and merged throttle and brake shutdown sense sheets into a single sheet - Shutdown_Sensors.kicad_sch.
Other:
- title: (none) -> Microcontroller - STM32G441CBT6
Changed lines of the file:
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@@
 	(generator_version "9.0")
 	(paper "A4")
+	(title_block
+		(title "Microcontroller - STM32G441CBT6")
+		(comment 1 "By Leo Liao")
+	)
 	(text "Power Supply Configuration\n(sec. 5.1.6 in datasheet)"
 		(exclude_from_sim no)

Commit message: Small tweaks, refer to DOC.pdf provided by Henry Tejada Deras on 01/25/2026
Parts:
- added C29: C_0.1uF, OEM:C_0603_1608Metric, symbol OEM:C_0.1uF_16V_0603
- R5: value R_200 -> R_1k; symbol OEM:R_200_0.1W_0603 -> OEM:R_1k_0.1W_0603; MPN WR06X2000FTL -> RMCF0603FT1K00 (or ERJ-3GEYJ102V)
Connections:
- net +3V3: now also C29.1
- net CAN_RX: now also U1.33 ((EVENTOUT/TIM1_BKIN2/TIM1_CH4/TIM4_CH1/FDCAN1_RX/COMP1_OUT/USART1_NSS/USART1_CTS/TIM1_CH1N/SPI2_MOSI/I2S2_SD/GPIO_EXTI11)PA11); no longer U1.45 ((EVENTOUT/SAI1_MCLK_A/TIM1_BKIN/TIM8_CH2/FDCAN1_RX/COMP1_OUT/USART3_RX/I2C1_SCL/SAI1_CK1/TIM4_CH3/TIM16_CH1/GPIO_EXTI8)PB8-BOOT0)
- net CAN_TX: now also U1.34 ((EVENTOUT/TIM1_ETR/TIM4_CH2/FDCAN1_TX/COMP2_OUT/USART1_RTS/USART1_DE/TIM1_CH2N/I2S_CKIN/TIM16_CH1/GPIO_EXTI12)PA12); no longer U1.46 ((EVENTOUT/SAI1_FS_A/TIM1_CH3N/TIM8_CH3/FDCAN1_TX/COMP2_OUT/USART3_TX/IR_OUT/I2C1_SDA/SAI1_D2/TIM4_CH4/TIM17_CH1/GPIO_EXTI9)PB9)
- net GND: now also C29.2
Other:
- moved on the sheet: C1, C2, C26, C28, C3, C4, C5, C6, C7, C8, D1, D14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
