File: vehicle/mkiii/hardware/integration/charging_board/J1772_V2.kicad_sch (KiCad schematic)
At the start: 81 parts, among them J10 J_Molex_Header_01x02_VT, J2 Conn_01x20_Socket, J5 J_Molex_Header_01x02_VT, J6 Conn_01x02_Socket, J7 J_Programming_Pin_Header, J8 J_Molex_Header_02x03_VT, J9 J_Molex_Header_01x02_VT, Q2 SSM3K333R,LF, Q3 SSM3K333R,LF, U1 TLV70450DBVR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

Commit message: Finished Draft 1 of Charging Board. Please Review. (WEIGHT REDUCTION)
Parts:
- added TP1: TP_SMD, OEM:TP_Hook_SMD, symbol OEM:TP_Hook_SMD
Connections:
- net +3V3 is gone; now on net +3.3V: F1.2
- net +3.3V: now also TP1.1
Changed lines of the file:
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@@
 	(rectangle
 		(start 15.24 172.72)
-		(end 135.89 220.98)
+		(end 146.05 220.98)
 		(stroke
 			(width 0)
@@
 	)
 	(junction
+		(at 130.81 193.04)
+		(diameter 0)
+		(color 0 0 0 0)
+	)
+	(junction
 		(at 335.28 153.67)
 		(diameter 0)
@@
 	(wire
 		(pts
+			(xy 130.81 193.04) (xy 130.81 190.5)
+		)
+		(stroke
+			(width 0)
+			(type default)
+		)
+	)
+	(wire
+		(pts
 			(xy 83.82 34.29) (xy 85.09 34.29)
 		)
@@
 	(wire
 		(pts
-			(xy 130.81 195.58) (xy 130.81 190.5)
+			(xy 130.81 195.58) (xy 130.81 193.04)
 		)
 		(stroke
@@
 		(dnp no)
 		(property "Reference" "C21"
-			(at 232.664 110.744 0)
+			(at 225.552 109.474 0)
 			(effects
 				(font
@@
 	)
 	(symbol
+		(lib_id "OEM:TP_Hook_SMD")
+		(at 132.08 193.04 270)
+		(unit 1)
+		(exclude_from_sim no)
+		(in_bom yes)
+		(on_board yes)
+		(dnp no)
+		(fields_autoplaced yes)
+		(property "Reference" "TP1"
+			(at 137.16 191.7699 90)
+			(effects
+				(font
+					(size 1.27 1.27)
+				)
+				(justify left)
+			)
+		)
+		(property "Value" "TP_SMD"
+			(at 137.16 194.3099 90)
+			(effects
+				(font
+					(size 1.27 1.27)
+				)
+				(justify left)
+			)
+		)
+		(property "Footprint" "OEM:TP_Hook_SMD"
+			(at 128.27 193.04 0)
+			(effects
+				(font
+					(size 1.27 1.27)
+				)
+				(hide yes)
+			)
+		)
+		(property "Datasheet" "https://www.mouser.com/datasheet/3/201/1/5019.PDF"
+			(at 132.08 193.04 0)
+			(effects
+				(font
+					(size 1.27 1.27)
+				)
+				(hide yes)
+			)
+		)
+		(property "Description" "Test Point SMD Hook"
+			(at 132.08 193.04 0)
+			(effects
+				(font
+					(size 1.27 1.27)
+				)
+				(hide yes)
+			)
+		)
+		(property "MPN" "5019"
+			(at 132.08 193.04 0)
+			(effects
+				(font
+					(size 1.27 1.27)
+				)
+				(hide yes)
+			)
+		)
+		(pin "1"
+		)
+		(instances
+			(project ""
+				(path "/8bf539d3-f4e7-408b-921d-45351bdd10f3"
+					(reference "TP1")
+					(unit 1)
+				)
+			)
+		)
+	)
+	(symbol
 		(lib_id "OEM:D_LED_White_0805")
 		(at 256.54 54.61 90)
@@
 	)
 	(symbol
+		(lib_id "power:+3.3V")
+		(at 130.81 190.5 0)
+		(unit 1)
+		(exclude_from_sim no)
+		(in_bom yes)
+		(on_board yes)
+		(dnp no)
+		(fields_autoplaced yes)
+		(property "Reference" "#PWR041"
+			(at 130.81 194.31 0)
+			(effects
+				(font
+					(size 1.27 1.27)
+				)
+				(hide yes)
+			)
+		)
+		(property "Value" "+3.3V"
+			(at 130.81 185.42 0)
+			(effects
+				(font
+					(size 1.27 1.27)
+				)
+			)
+		)
+		(property "Footprint" ""
+			(at 130.81 190.5 0)
+			(effects
+				(font
+					(size 1.27 1.27)
+				)
+				(hide yes)
+			)
+		)
+		(property "Datasheet" ""
+			(at 130.81 190.5 0)
+			(effects
+				(font
+					(size 1.27 1.27)
+				)
+				(hide yes)
+			)
+		)
+		(property "Description" "Power symbol creates a global label with name \"+3.3V\""
+			(at 130.81 190.5 0)
+			(effects
+				(font
+					(size 1.27 1.27)
+				)
+				(hide yes)
+			)
+		)
+		(pin "1"
+		)
+		(instances
+			(project ""
+				(path "/8bf539d3-f4e7-408b-921d-45351bdd10f3"
+					(reference "#PWR041")
+					(unit 1)
+				)
+			)
+		)
+	)
+	(symbol
 		(lib_name "GND_33")
 		(lib_id "power:GND")
@@
 					(unit 1)
 				)
-			)
-		)
-	)
-	(symbol
-		(lib_id "power:+3V3")
-		(at 130.81 190.5 0)
-		(unit 1)
-		(exclude_from_sim no)
-		(in_bom yes)
-		(on_board yes)
-		(dnp no)
-		(fields_autoplaced yes)
-		(property "Reference" "#PWR041"
-			(at 130.81 194.31 0)
-			(effects
-				(font
-					(size 1.27 1.27)
-				)
-				(hide yes)
-			)
-		)
-		(property "Value" "+3V3"
-			(at 130.81 185.42 0)
-			(effects
-				(font
-					(size 1.27 1.27)
-				)
-			)
-		)
-		(property "Footprint" ""
-			(at 130.81 190.5 0)
-			(effects
-				(font
-					(size 1.27 1.27)
-				)
-				(hide yes)
-			)
-		)
-		(property "Datasheet" ""
-			(at 130.81 190.5 0)
-			(effects
-				(font
-					(size 1.27 1.27)
-				)
-				(hide yes)
-			)
-		)
-		(property "Description" "Power symbol creates a global label with name \"+3V3\""
-			(at 130.81 190.5 0)
-			(effects
-				(font
-					(size 1.27 1.27)
-				)
-				(hide yes)
-			)
-		)
-		(pin "1"
-		)
-		(instances
-			(project ""
-				(path "/8bf539d3-f4e7-408b-921d-45351bdd10f3"
-					(reference "#PWR041")
-					(unit 1)
-				)
