File: vehicle/mkiii/hardware/integration/BMS_Coew/bms_core.kicad_pcb (KiCad board)
At the start: 4 copper layers, 101.4 x 25.1 mm, 88 parts, among them J2 CONN_02x03, J3 MicroFit_RA_2, J4 J_Programming_Pin_Header, J5 J_PCIe_x1, K1 Relay_G5Q-1A4-DC5, Q1 SSM3K333R, T1 HM2112ZNLT, U10 STM32G441KBT6, U11 MCP2561-E_SN, U3 LTC6820HMS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

Commit message: Final version I think
Parts:
- moved REF** 85.7 mm to (82.2, 196.3)
- moved kibuzzard-673AE93C 85.7 mm to (71.5, 199.0)
- moved kibuzzard-673AE955 85.7 mm to (71.5, 196.2)
- moved kibuzzard-673AE966 85.7 mm to (73.5, 193.4)
- moved C9 2.61 mm to (232.5, 146.0), turned to 180 degrees
- moved GND_SHORT 0.59 mm to (212.5, 145.0)
- moved BSPD1 0.20 mm to (225.2, 154.5)
- moved U4 0.16 mm to (232.1, 148.6)
- moved U5 0.06 mm to (209.3, 149.5)
- turned IM1 to 0 degrees
- turned IP1 to 0 degrees
- renumbered DIFF_AMP to TP10, CURRENT_TRIP to TP4, VGND to V_GND
Routing:
- net GND: track 76.1 -> 78.7 mm
- net /Heartbeat: track 25.4 -> 23.3 mm
- net /BSPD Current Sensor Trigger/CURRENT_TRIP: track 6.43 -> 4.51 mm
- net /SHDN_OUT: track 53.3 -> 54.9 mm
- net Net-(U8--): track 4.65 -> 6.06 mm
- net /BSPD Current Sensor Trigger/GND_SHORT: track 10.3 -> 11.4 mm
- net /CSC_Comms: track 25.3 -> 24.3 mm
- net Net-(U8-+): track 3.16 -> 3.82 mm
- net /Error: track 28.9 -> 28.4 mm
- net +5V: track 46.1 -> 46.0 mm, vias 14 -> 13
- net /NRST: vias 3 -> 2
