File: vehicle/mkiii/hardware/integration/bms_core/m_2_connector.kicad_sch (KiCad schematic)
At the start: 1 part, among them J5 J_PCIe_x1

Commit message: Changes according to feedback
Parts:
- added C1: C_0.1uF_16V, OEM:C_0603_1608Metric, symbol OEM:C_0.1uF_16V_0603
- added U1: MCP6001, Package_TO_SOT_SMD:SOT-353_SC-70-5, symbol OEM:MCP6001
Connections:
- net +5V: now also C1.2, U1.5 (V+)
- net GND: now also C1.1, U1.2 (V-)
- net VOUT_CURRENT_SENSE: now also U1.1, U1.4 (-); no longer J5.B8 (io_5)
- new net: J5.B8 (io_5), U1.3 (+)
Other:
- note added: "+5V +3V3 and GND come from the Service Section Motherboard."
- note removed: "+5V and GND come from the Service Section Motherboard."

Commit message: Added Subteam Logo, Production Files, and readded isoSPI debugging header.
Changed lines of the file:
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@@
-	)
-	(label "GND"
-		(at 153.67 100.33 180)
-		(effects
-			(font
-				(size 1.27 1.27)
-			)
-			(justify right bottom)
-		)
 	)
 	(label "GND"
@@
 		(dnp no)
 		(fields_autoplaced yes)
-		(property "Reference" "#PWR?"
+		(property "Reference" "#PWR0162"
 			(at 148.59 80.01 0)
 			(effects
@@
 			(project ""
 				(path "/19b2a9f9-0be6-4bde-80c5-cbc5126d55d5/8857e594-f9a2-447b-85c9-7fce31d1bf44"
-					(reference "#PWR?")
+					(reference "#PWR0162")
 					(unit 1)
 				)
@@
 		(on_board yes)
 		(dnp no)
-		(property "Reference" "#PWR?"
+		(property "Reference" "#PWR0164"
 			(at 148.59 106.68 0)
 			(effects
@@
 			(project "bms_core"
 				(path "/19b2a9f9-0be6-4bde-80c5-cbc5126d55d5/8857e594-f9a2-447b-85c9-7fce31d1bf44"
-					(reference "#PWR?")
+					(reference "#PWR0164")
 					(unit 1)
 				)
@@
 		(dnp no)
 		(fields_autoplaced yes)
-		(property "Reference" "#PWR?"
+		(property "Reference" "#PWR0160"
 			(at 91.44 66.04 0)
 			(effects
@@
 			(project ""
 				(path "/19b2a9f9-0be6-4bde-80c5-cbc5126d55d5/8857e594-f9a2-447b-85c9-7fce31d1bf44"
-					(reference "#PWR?")
+					(reference "#PWR0160")
 					(unit 1)
 				)
@@
 		(dnp no)
 		(fields_autoplaced yes)
-		(property "Reference" "#PWR?"
+		(property "Reference" "#PWR0163"
 			(at 160.02 82.55 0)
 			(effects
@@
 			(project ""
 				(path "/19b2a9f9-0be6-4bde-80c5-cbc5126d55d5/8857e594-f9a2-447b-85c9-7fce31d1bf44"
-					(reference "#PWR?")
+					(reference "#PWR0163")
 					(unit 1)
 				)
@@
 		(dnp no)
 		(fields_autoplaced yes)
-		(property "Reference" "#PWR?"
+		(property "Reference" "#PWR0161"
 			(at 87.63 66.04 0)
 			(effects
@@
 			(project ""
 				(path "/19b2a9f9-0be6-4bde-80c5-cbc5126d55d5/8857e594-f9a2-447b-85c9-7fce31d1bf44"
-					(reference "#PWR?")
+					(reference "#PWR0161")
 					(unit 1)
 				)
