File: vehicle/mkiii/hardware/lv/VCU/microcontroller.kicad_sch (KiCad schematic)
At the start: 36 parts, among them J1 J_Programming_Pin_Header, U1 STM32G441CBT6, U12 MCP2561-E_SN, Y1 X_16MHz_18pF

Commit message: Layout completed, review required
Parts:
- added TP2: 3V3, OEM:TP_Hook_SMD, symbol OEM:TP_Hook_SMD
- D5: renamed from D14; value HEARTBEAT -> THROTTLE_DISABLE
- D8: renamed from D7; value MISO -> NRST
- D9: renamed from D8; value MOSI -> SWDIO
- renumbered C29 to C1, C8 to C10, C26 to C11, C1 to C3, C3 to C5, C5 to C6, C28 to C7, C7 to C8, C6 to C9, D5 to D6, D6 to D7, R39 to R10, R49 to R5, R5 to R6, R6 to R7, R7 to R8, R8 to R9, TP2 to TP3, U12 to U2
Connections:
- net HEARTBEAT is gone; now on net HEARTBEAT_LED: U1.43 ((EVENTOUT/SAI1_FS_B/LPTIM1_ETR/TIM8_BKIN2/COMP4_OUT/USART1_TX/TIM8_ETR/TIM8_CH1/TIM4_CH1/TIM16_CH1N/GPIO_EXTI6)PB6)
- net +3V3: now also TP2.1; no longer U1.1 (VBAT)
- no-connect marks 1 -> 23
Other:
- note added: "5V, 3V3, and Ground Lines Test Points"
- note removed: "5V and Ground Lines Test Points"
- moved on the sheet: TP1
