File: vehicle/mkviii/hardware/hv/power_thermistor/power_thermistor.kicad_pcb (KiCad board)
At the start: 4 copper layers, 400.9 x 174.3 mm, 124 parts, among them J1 T2M-110-01-X-D-TH-WT, J10 Battery Cell Spot Weld, J11 Battery Cell Spot Weld, J12 Battery Cell Spot Weld, J13 Battery Cell Spot Weld, J14 Battery Cell Spot Weld, J15 Battery Cell Spot Weld, J16 Battery Cell Spot Weld, J17 Battery Cell Spot Weld, J18 Battery Cell Spot Weld, J19 Battery Cell Spot Weld, J2 J_Molex_Header_01x02_VT, J20 J_Redcube, J22 Battery Cell Spot Weld, J23 J_Redcube, J3 T2M-110-01-X-D-TH-WT, J4 T2M-110-01-X-D-TH-WT, J5 Battery Cell Spot Weld, J50 Battery Cell Spot Weld, J51 Battery Cell Spot Weld, J6 J_Molex_Header_01x02_VT, J7 Battery Cell Spot Weld, J8 Battery Cell Spot Weld, J9 Battery Cell Spot Weld, U1 DS18B20U

Commit message: Modified 1-Wire Traces; Added Final Production Files
Routing:
- net Net-(U1-GND): track 301.5 -> 396.8 mm
- net Net-(U1-DQ): track 298.9 -> 385.4 mm, vias 3 -> 1
Changed lines of the file:
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@@
 			(at 0 -2 180)
 			(layer "B.SilkS")
+			(hide yes)
 			(effects
 				(font
@@
 			(at -13.72 5.135 180)
 			(layer "B.SilkS")
+			(hide yes)
 			(effects
 				(font
@@
 			(at -5.084 1.325 180)
 			(layer "B.SilkS")
+			(hide yes)
 			(effects
 				(font
@@
 			(at 0 -2 180)
 			(layer "B.SilkS")
+			(hide yes)
 			(effects
 				(font
@@
 			(at -13.72 5.135 180)
 			(layer "B.SilkS")
+			(hide yes)
 			(effects
 				(font
@@
 	)
 	(via
-		(at 222.25 158.17)
+		(at 221.751523 158.17)
 		(size 0.6)
 		(drill 0.3)
@@
 	)
 	(segment
-		(start 222.25 158.512622)
-		(end 222.643586 158.906208)
+		(start 227.063186 160.856928)
+		(end 226.056786 160.856928)
 		(width 0.2)
 		(layer "B.Cu")
@@
 	)
 	(segment
-		(start 227.063186 160.856928)
-		(end 226.056786 160.856928)
+		(start 222.25 158.512622)
+		(end 222.643586 158.906208)
 		(width 0.2)
 		(layer "B.Cu")
@@
 	)
 	(segment
-		(start 222.25 158.17)
+		(start 221.751523 158.17)
+		(end 222.094145 158.512622)
+		(width 0.2)
+		(layer "B.Cu")
+		(net 68)
+	)
+	(segment
+		(start 222.094145 158.512622)
 		(end 222.25 158.512622)
 		(width 0.2)
@@
 	(segment
 		(start 221.751523 158.17)
-		(end 222.25 158.17)
+		(end 222.091523 158.51)
+		(width 0.2)
+		(layer "In1.Cu")
+		(net 68)
+	)
+	(segment
+		(start 268.37 23.63)
+		(end 233.172562 58.827438)
+		(width 0.2)
+		(layer "In1.Cu")
+		(net 68)
+	)
+	(segment
+		(start 269.13 23.63)
+		(end 270.21 23.63)
 		(width 0.2)
 		(layer "In1.Cu")
@@
 	(segment
 		(start 220.5 63.56)
-		(end 220.55 63.56)
+		(end 199.64 42.7)
 		(width 0.2)
 		(layer "In1.Cu")
@@
 	)
 	(segment
-		(start 220.5 156.918477)
-		(end 220.5 63.56)
+		(start 231.2 158.51)
+		(end 233.172562 156.537438)
 		(width 0.2)
 		(layer "In1.Cu")
@@
 	)
 	(segment
-		(start 230.56 60.69)
-		(end 267.62 23.63)
+		(start 233.172562 58.827438)
+		(end 233.172562 154.908609)
 		(width 0.2)
 		(layer "In1.Cu")
@@
 	)
 	(segment
-		(start 269.13 23.63)
-		(end 270.21 23.63)
+		(start 233.173471 154.909579)
+		(end 233.172562 154.937433)
 		(width 0.2)
 		(layer "In1.Cu")
@@
 	)
 	(segment
-		(start 220.5 63.56)
-		(end 199.64 42.7)
+		(start 233.172562 156.537438)
+		(end 233.172562 154.908609)
 		(width 0.2)
 		(layer "In1.Cu")
@@
 	)
 	(segment
-		(start 220.55 63.56)
-		(end 223.42 60.69)
+		(start 221.751523 158.17)
+		(end 220.5 156.918477)
 		(width 0.2)
 		(layer "In1.Cu")
@@
 	)
 	(segment
-		(start 267.62 23.63)
-		(end 270.21 23.63)
+		(start 270.21 23.63)
+		(end 268.37 23.63)
 		(width 0.2)
 		(layer "In1.Cu")
@@
 	(segment
 		(start 220.5 156.918477)
-		(end 221.751523 158.17)
+		(end 220.5 63.56)
+		(width 0.2)
+		(layer "In1.Cu")
+		(net 68)
+	)
+	(segment
+		(start 222.091523 158.51)
+		(end 231.2 158.51)
 		(width 0.2)
 		(layer "In1.Cu")
@@
 	)
 	(segment
-		(start 223.42 60.69)
-		(end 230.56 60.69)
+		(start 233.172562 154.908609)
+		(end 233.173471 154.909579)
 		(width 0.2)
 		(layer "In1.Cu")
@@
 	)
 	(via
-		(at 221.68 65.53)
+		(at 228.49 159.13)
 		(size 0.6)
 		(drill 0.3)
@@
 		(net 69)
 	)
-	(via
-		(at 228.35 158.84)
-		(size 0.6)
-		(drill 0.3)
-		(layers "F.Cu" "B.Cu")
-		(net 69)
-	)
-	(via
-		(at 219.2 64.43)
-		(size 0.6)
-		(drill 0.3)
-		(layers "F.Cu" "B.Cu")
+	(segment
+		(start 228.2 158.84)
+		(end 227.129394 158.84)
+		(width 0.2)
+		(layer "B.Cu")
 		(net 69)
 	)
 	(segment
-		(start 220.3 65.53)
-		(end 219.2 64.43)
+		(start 228.49 159.13)
+		(end 228.2 158.84)
 		(width 0.2)
 		(layer "B.Cu")
@@
 	)
 	(segment
-		(start 228.35 158.84)
-		(end 227.129394 158.84)
+		(start 227.15254 158.995562)
+		(end 227.063186 158.906208)
 		(width 0.2)
 		(layer "B.Cu")
@@
 	)
 	(segment
-		(start 221.68 65.53)
-		(end 220.3 65.53)
+		(start 233.578662 154.757029)
+		(end 233.573532 154.751553)
 		(width 0.2)
-		(layer "B.Cu")
+		(layer "In1.Cu")
 		(net 69)
 	)
 	(segment
-		(start 227.15254 158.995562)
-		(end 227.063186 158.906208)
+		(start 233.572562 156.703123)
+		(end 233.572562 155.076235)
 		(width 0.2)
-		(layer "B.Cu")
+		(layer "In1.Cu")
 		(net 69)
 	)
 	(segment
-		(start 122.28 44.3)
-		(end 104.61 26.63)
+		(start 233.572562 154.742923)
+		(end 233.572562 63.267438)
 		(width 0.2)
 		(layer "In1.Cu")
@@
 	)
 	(segment
-		(start 233.6 65.63)
-		(end 270.21 29.02)
+		(start 220.1 157.37)
+		(end 220.1 65.93)
 		(width 0.2)
 		(layer "In1.Cu")
@@
 	)
 	(segment
-		(start 198.47 44.3)
-		(end 122.28 44.3)
+		(start 233.572562 155.076235)
+		(end 233.573532 155.075265)
 		(width 0.2)
 		(layer "In1.Cu")
@@
 	)
 	(segment
-		(start 221.68 65.53)
-		(end 221.78 65.63)
+		(start 221.86 159.13)
+		(end 220.1 157.37)
 		(width 0.2)
 		(layer "In1.Cu")
@@
 	)
 	(segment
-		(start 233.6 67.75)
-		(end 233.6 156.824255)
+		(start 220.1 65.93)
+		(end 198.47 44.3)
 		(width 0.2)
 		(layer "In1.Cu")
@@
 	)
 	(segment
-		(start 221.78 65.63)
-		(end 231.48 65.63)
+		(start 233.573532 154.914229)
+		(end 233.578662 154.757029)
 		(width 0.2)
 		(layer "In1.Cu")
@@
 	)
 	(segment
-		(start 231.48 65.63)
-		(end 233.6 67.75)
+		(start 233.573532 154.751553)
+		(end 233.573532 154.743893)
 		(width 0.2)
 		(layer "In1.Cu")
@@
 	)
 	(segment
-		(start 231.584255 158.84)
-		(end 228.35 158.84)
+		(start 228.49 159.13)
+		(end 221.86 159.13)
 		(width 0.2)
 		(layer "In1.Cu")
@@
 	)
 	(segment
-		(start 270.21 29.02)
-		(end 270.21 26.63)
+		(start 122.28 44.3)
+		(end 104.61 26.63)
 		(width 0.2)
 		(layer "In1.Cu")
@@
 	)
 	(segment
-		(start 233.6 67.75)
-		(end 233.6 65.63)
+		(start 231.145686 159.13)
+		(end 233.572562 156.703123)
 		(width 0.2)
 		(layer "In1.Cu")
@@
 	)
 	(segment
-		(start 233.6 156.824255)
-		(end 231.584255 158.84)
+		(start 233.573532 154.743893)
+		(end 233.572562 154.742923)
 		(width 0.2)
 		(layer "In1.Cu")
@@
 	)
 	(segment
-		(start 219.2 64.43)
-		(end 218.6 64.43)
+		(start 233.573532 155.075265)
+		(end 233.573532 154.914229)
 		(width 0.2)
 		(layer "In1.Cu")
@@
 	)
 	(segment
-		(start 218.6 64.43)
-		(end 198.47 44.3)
+		(start 198.47 44.3)
+		(end 122.28 44.3)
+		(width 0.2)
+		(layer "In1.Cu")
+		(net 69)
+	)
+	(segment
+		(start 228.49 159.13)
+		(end 231.145686 159.13)
+		(width 0.2)
+		(layer "In1.Cu")
+		(net 69)
+	)
+	(segment
+		(start 233.572562 63.267438)
+		(end 270.21 26.63)
 		(width 0.2)
 		(layer "In1.Cu")
