File: vehicle/mkviii/hardware/lv/CarStat/buck_converters.kicad_sch (KiCad schematic)
At the start: 14 parts, among them U3 AD62305WU-7, U4 AP63203WU-7

Commit message: Layout v2
Parts:
- removed C10, C11: C_10uF_10V, OEM:C_0603_1608Metric, symbol OEM:C_10uF_10V_0603
- added C10, C11: C_10uF_35V, OEM:C_0603_1608Metric, symbol OEM:C_10uF_35V_0603
Connections:
- net 12V: now also C10.1, C11.1
- net GND: now also C10.2, C11.2
