File: vehicle/mkviii/hardware/lv/CarStat/status_leds.kicad_sch (KiCad schematic)
At the start: 38 parts

Commit message: Layout v2
Parts:
- removed D13: LED, OEM:D_0805_2012Metric, symbol OEM:D_LED_White_0805
- removed R13: R_1k_0.1W, OEM:R_0603_1608Metric, symbol OEM:R_1k_0.1W_0603
Other:
- note removed: "Shutdown Circuit Closed"
