File: vehicle/mkviii/hardware/lv/CarStat/CarStat.kicad_sch (KiCad schematic)
At the start: 34 parts, among them J1 430450412, J2 J_Programming_Pin_Header, U1 MCP2561-E_SN, U2 STM32G441KBT6, U7 MCP6001T-I/LT, Y1 X_16MHz_18pF

Commit message: Layout v2
Parts:
- removed C19: C_22uF_25V, OEM:C_1206_3216Metric, symbol OEM:C_22uF_25V_1206
- added C18: C_10uF_35V, OEM:C_0603_1608Metric, symbol OEM:C_10uF_35V_0603
- added D13: LED, OEM:D_0805_2012Metric, symbol OEM:D_LED_White_0805
- added R13: R_1k_0.1W, OEM:R_0603_1608Metric, symbol OEM:R_1k_0.1W_0603
Connections:
- net SHDN.FULL_C is gone; now on net SHDN.AIR-N: U2.19 ((TIM2_CH3/TIM15_BKIN/USART1_TX/GPIO_EXTI9)PA9)
- net +12V: now also C18.1, R13.1
- net GND: now also C18.2, D13.1 (K)
- net HEARTBEAT: now also U2.2 (PF0-OSC_IN)
- net SHDN.AIR-N: no longer U2.18 ((TIM4_ETR/USART1_CK/GPIO_EXTI8)PA8)
- net SHDN.AIR-P: now also U2.3 (PF1-OSC_OUT); no longer U2.2 (PF0-OSC_IN)
- net SHDN.BMS: now also U2.7 ((TIM15_CH1/USART2_TX/TIM2_CH3/GPIO_EXTI2/ADC1_IN3)PA2*); no longer U2.6 ((TIM15_CH1N/TIM2_CH2/GPIO_EXTI1/ADC2_IN2/ADC1_IN2)PA1*)
- net SHDN.BOTS: now also U2.13 ((TIM3_CH3/GPIO_EXTI0/ADC1_IN15)PB0*); no longer U2.12 ((TIM3_CH2/TIM17_CH1/GPIO_EXTI7/ADC2_IN4)PA7*)
- net SHDN.BSPD: now also U2.12 ((TIM3_CH2/TIM17_CH1/GPIO_EXTI7/ADC2_IN4)PA7*); no longer U2.11 ((TIM3_CH1/TIM16_CH1/GPIO_EXTI6/ADC2_IN3)PA6*)
- net SHDN.EMETER: now also U2.10 ((TIM2_ETR/TIM2_CH1/GPIO_EXTI5/ADC2_IN13)PA5*); no longer U2.9 ((USART2_CK/TIM3_CH2/GPIO_EXTI4/ADC2_IN17)PA4*)
- net SHDN.HVD: now also U2.11 ((TIM3_CH1/TIM16_CH1/GPIO_EXTI6/ADC2_IN3)PA6*); no longer U2.10 ((TIM2_ETR/TIM2_CH1/GPIO_EXTI5/ADC2_IN13)PA5*)
- net SHDN.IMD: now also U2.6 ((TIM15_CH1N/TIM2_CH2/GPIO_EXTI1/ADC2_IN2/ADC1_IN2)PA1*); no longer U2.5 ((TIM2_ETR/TIM2_CH1/GPIO_EXTI0/ADC2_IN1/ADC1_IN1)PA0*)
- net SHDN.IS: now also U2.18 ((TIM4_ETR/USART1_CK/GPIO_EXTI8)PA8); no longer U2.13 ((TIM3_CH3/GPIO_EXTI0/ADC1_IN15)PB0*)
- net SHDN.MPC: now also U2.8 ((TIM15_CH2/USART2_RX/TIM2_CH4/GPIO_EXTI3/ADC1_IN4)PA3*); no longer U2.7 ((TIM15_CH1/USART2_TX/TIM2_CH3/GPIO_EXTI2/ADC1_IN3)PA2*)
- net SHDN.TSMP: now also U2.9 ((USART2_CK/TIM3_CH2/GPIO_EXTI4/ADC2_IN17)PA4*); no longer U2.8 ((TIM15_CH2/USART2_RX/TIM2_CH4/GPIO_EXTI3/ADC1_IN4)PA3*)
- net SHDN.TSMS: now also U2.5 ((TIM2_ETR/TIM2_CH1/GPIO_EXTI0/ADC2_IN1/ADC1_IN1)PA0*); no longer U2.3 (PF1-OSC_OUT)
- new net: D13.2 (A), R13.2
Other:
- sheet Status LEDs ports: added none; removed F_SS_C
- moved on the sheet: D5, R6

Commit message: Layout Draft 3
Connections:
- net +12V: now also F3.2; no longer F3.1
- net +3V3: now also U7.5 (V+)
- net +5V: no longer U7.5 (V+)
- net Debug1: now also U2.26 ((TIM3_ETR/SPI1_SCK/TIM4_ETR/TIM2_CH2/GPIO_EXTI3)PB3); no longer U2.29 ((TIM4_CH1/TIM16_CH1N/GPIO_EXTI6)PB6)
- net Debug2: now also U2.27 ((TIM17_BKIN/SPI1_MISO/TIM3_CH1/TIM16_CH1/GPIO_EXTI4)PB4); no longer U2.28 ((TIM17_CH1/SPI1_MOSI/TIM3_CH2/TIM16_BKIN/GPIO_EXTI5)PB5)
- net Debug3: now also U2.28 ((TIM17_CH1/SPI1_MOSI/TIM3_CH2/TIM16_BKIN/GPIO_EXTI5)PB5); no longer U2.27 ((TIM17_BKIN/SPI1_MISO/TIM3_CH1/TIM16_CH1/GPIO_EXTI4)PB4)
- net ESTOP.DRIVER: now also U2.29 ((TIM4_CH1/TIM16_CH1N/GPIO_EXTI6)PB6); no longer U2.26 ((TIM3_ETR/SPI1_SCK/TIM4_ETR/TIM2_CH2/GPIO_EXTI3)PB3)
- net ESTOP.LEFT: now also U2.30 ((TIM3_CH4/TIM4_CH2/TIM17_CH1N/GPIO_EXTI7)PB7); no longer U2.25 ((TIM2_ETR/TIM2_CH1/GPIO_EXTI15)PA15)
- net ESTOP.RIGHT: now also U2.31 ((TIM4_CH3/TIM16_CH1/GPIO_EXTI8)PB8-BOOT0); no longer U2.20 ((TIM2_CH4/USART1_RX/TIM17_BKIN/GPIO_EXTI10)PA10)
- net HEARTBEAT: now also U2.25 ((TIM2_ETR/TIM2_CH1/GPIO_EXTI15)PA15); no longer U2.2 (PF0-OSC_IN)
- net SHDN.AIR-N: now also U2.8 ((TIM15_CH2/USART2_RX/TIM2_CH4/GPIO_EXTI3/ADC1_IN4)PA3*); no longer U2.19 ((TIM2_CH3/TIM15_BKIN/USART1_TX/GPIO_EXTI9)PA9)
- net SHDN.AIR-P: now also U2.7 ((TIM15_CH1/USART2_TX/TIM2_CH3/GPIO_EXTI2/ADC1_IN3)PA2*); no longer U2.3 (PF1-OSC_OUT)
- net SHDN.BMS: now also U2.12 ((TIM3_CH2/TIM17_CH1/GPIO_EXTI7/ADC2_IN4)PA7*); no longer U2.7 ((TIM15_CH1/USART2_TX/TIM2_CH3/GPIO_EXTI2/ADC1_IN3)PA2*)
- net SHDN.BOTS: now also U2.19 ((TIM2_CH3/TIM15_BKIN/USART1_TX/GPIO_EXTI9)PA9); no longer U2.13 ((TIM3_CH3/GPIO_EXTI0/ADC1_IN15)PB0*)
- net SHDN.BSPD: now also U2.18 ((TIM4_ETR/USART1_CK/GPIO_EXTI8)PA8); no longer U2.12 ((TIM3_CH2/TIM17_CH1/GPIO_EXTI7/ADC2_IN4)PA7*)
- net SHDN.EMETER: now also U2.9 ((USART2_CK/TIM3_CH2/GPIO_EXTI4/ADC2_IN17)PA4*); no longer U2.10 ((TIM2_ETR/TIM2_CH1/GPIO_EXTI5/ADC2_IN13)PA5*)
- net SHDN.HVD: now also U2.13 ((TIM3_CH3/GPIO_EXTI0/ADC1_IN15)PB0*); no longer U2.11 ((TIM3_CH1/TIM16_CH1/GPIO_EXTI6/ADC2_IN3)PA6*)
- net SHDN.IMD: now also U2.5 ((TIM2_ETR/TIM2_CH1/GPIO_EXTI0/ADC2_IN1/ADC1_IN1)PA0*); no longer U2.6 ((TIM15_CH1N/TIM2_CH2/GPIO_EXTI1/ADC2_IN2/ADC1_IN2)PA1*)
- net SHDN.IS: now also U2.20 ((TIM2_CH4/USART1_RX/TIM17_BKIN/GPIO_EXTI10)PA10); no longer U2.18 ((TIM4_ETR/USART1_CK/GPIO_EXTI8)PA8)
- net SHDN.MPC: now also U2.11 ((TIM3_CH1/TIM16_CH1/GPIO_EXTI6/ADC2_IN3)PA6*); no longer U2.8 ((TIM15_CH2/USART2_RX/TIM2_CH4/GPIO_EXTI3/ADC1_IN4)PA3*)
- net SHDN.TSMP: now also U2.10 ((TIM2_ETR/TIM2_CH1/GPIO_EXTI5/ADC2_IN13)PA5*); no longer U2.9 ((USART2_CK/TIM3_CH2/GPIO_EXTI4/ADC2_IN17)PA4*)
- net SHDN.TSMS: now also U2.6 ((TIM15_CH1N/TIM2_CH2/GPIO_EXTI1/ADC2_IN2/ADC1_IN2)PA1*); no longer U2.5 ((TIM2_ETR/TIM2_CH1/GPIO_EXTI0/ADC2_IN1/ADC1_IN1)PA0*)
- net +12VIN: now reaches J1.1
- net +12VIN: now also F3.1; no longer F3.2
- net at C8.1, Y1.3: now also U2.2 (PF0-OSC_IN); no longer U2.30 ((TIM3_CH4/TIM4_CH2/TIM17_CH1N/GPIO_EXTI7)PB7)
- net at C9.2, Y1.1: now also U2.3 (PF1-OSC_OUT); no longer U2.31 ((TIM4_CH3/TIM16_CH1/GPIO_EXTI8)PB8-BOOT0)
Other:
- moved on the sheet: C8, C9, F3, Y1
