File: vehicle/mkviii/hardware/lv/CarStat/CarStat.kicad_pcb (KiCad board)
At the start: 2 copper layers, 90 x 47.5 mm, 86 parts, among them J1 430450412, J2 J_Programming_Pin_Header, U1 MCP2561-E_SN, U2 STM32G441KBT6, U3 AD62305WU-7, U4 AP63203WU-7, U7 MCP6001T-I/LT, Y1 X_16MHz_18pF

Commit message: Layout v2
Parts:
- removed C19: C_22uF_25V, OEM:C_1206_3216Metric
- added C18: C_10uF_35V, OEM:C_0603_1608Metric, F.Cu at (193.6, 84.2)
- C10, C11: value C_10uF_10V -> C_10uF_35V
- moved R13 54.5 mm to (201.2, 113.9), turned to -90 degrees
- moved D13 49.3 mm to (203.1, 113.9), turned to -90 degrees
- moved TP5 34.1 mm to (186.7, 87.1)
- moved TP6 32.7 mm to (181.7, 87.1)
- moved R4 30.4 mm to (207.0, 82.6), turned to 90 degrees
- moved TP3 28.6 mm to (193.2, 93.8)
- moved D4 27.9 mm to (205.0, 82.6), turned to 90 degrees
- moved TP2 24.9 mm to (193.8, 105.5)
- moved R2 23.2 mm to (196.8, 93.7), turned to -90 degrees
- moved U7 22.7 mm to (202.4, 82.7), turned to 90 degrees
- moved R3 22.5 mm to (200.2, 83.0), turned to 90 degrees
- moved D2 20.9 mm to (198.8, 93.8), turned to -90 degrees
- moved D3 20.5 mm to (198.2, 83.0), turned to 90 degrees
- moved TP4 16.6 mm to (197.1, 114.7)
- moved R1 11.2 mm to (197.2, 105.4), turned to -90 degrees
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Connections:
- R13 pad 1: /SHDN.FULL_C -> +12V
- U2 pad 10: /SHDN.HVD -> /SHDN.EMETER
- U2 pad 11: /SHDN.BSPD -> /SHDN.HVD
- U2 pad 12: /SHDN.BOTS -> /SHDN.BSPD
- U2 pad 13: /SHDN.IS -> /SHDN.BOTS
- U2 pad 18: /SHDN.AIR-N -> /SHDN.IS
- U2 pad 19: /SHDN.FULL_C -> /SHDN.AIR-N
- U2 pad 2: /SHDN.AIR-P -> /HEARTBEAT
- U2 pad 3: /SHDN.TSMS -> /SHDN.AIR-P
- U2 pad 5: /SHDN.IMD -> /SHDN.TSMS
- U2 pad 6: /SHDN.BMS -> /SHDN.IMD
- U2 pad 7: /SHDN.MPC -> /SHDN.BMS
- U2 pad 8: /SHDN.TSMP -> /SHDN.MPC
- U2 pad 9: /SHDN.EMETER -> /SHDN.TSMP
Routing:
- net +12V: track 71.2 -> 3.09 mm
- net +5V: track 65.9 -> 2.58 mm, vias 2 -> 0
- net +3V3: track 82.9 -> 30.0 mm
- net /SHDN.FULL_C: track 52.7 -> 0.00 mm, vias 2 -> 0
- net /CAN+: track 68.9 -> 17.6 mm, vias 2 -> 0
- net /CAN-: track 65.5 -> 20.9 mm, vias 2 -> 0
- net /SWDIO: track 46.0 -> 13.5 mm, vias 2 -> 1
- net GND: track 34.8 -> 15.3 mm, vias 15 -> 50
- net /NRST: track 44.0 -> 34.0 mm
- net /HEARTBEAT: track 0.00 -> 9.89 mm
- net Net-(U4-FB): track 26.2 -> 16.8 mm
- net Net-(U2-(TIM4_CH3/TIM16_CH1/GPIO_EXTI8)PB8-BOOT0): track 17.3 -> 8.69 mm
- net Net-(U3-SW): track 8.22 -> 0.00 mm
- net Net-(U3-FB): track 22.1 -> 14.2 mm
- net Net-(U4-SW): track 7.56 -> 1.96 mm
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- added copper zone on F.Cu, net +12V
- added copper zone on F.Cu, net +3V3
- added copper zone on F.Cu, net +5V
- added copper zone on F.Cu, net Net-(U3-FB)
- added copper zone on F.Cu, net Net-(U3-SW)
- added copper zone on F.Cu, net Net-(U4-FB)
- added copper zone on F.Cu, net Net-(U4-SW)
Other:
- board text added: "HEARTBEAT"
- board text removed: "CIRCUIT CLOSED"
- board text removed: "HB"

Commit message: Layout Draft 3
Parts:
- moved F2 38.9 mm to (203.2, 76.4), turned to 90 degrees
- moved TP1 38.8 mm to (216.6, 76.6), turned to -90 degrees
- moved R3 38.2 mm to (218.4, 116.5), turned to 0 degrees
- moved D3 37.6 mm to (218.3, 114.7), turned to 0 degrees
- moved J2 36.8 mm to (204.8, 114.6)
- moved D13 36.5 mm to (183.0, 83.5), turned to 0 degrees
- moved U7 35.4 mm to (214.8, 115.8), turned to 0 degrees
- moved C15 34.4 mm to (196.7, 82.5)
- moved R13 33.9 mm to (183.2, 85.2), turned to 0 degrees
- moved TP2 33.4 mm to (210.5, 76.6), turned to -90 degrees
- moved TP4 32.9 mm to (187.3, 83.3), turned to 0 degrees
- moved C12 32.1 mm to (192.8, 76.9)
- moved U4 32.1 mm to (192.2, 79.5)
- moved C11 32.1 mm to (191.9, 82.1)
- moved L1 31.9 mm to (198.0, 77.6)
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Connections:
- C8 pad 1: Net-(U2-(TIM3_CH4/TIM4_CH2/TIM17_CH1N/GPIO_EXTI7)PB7) -> Net-(U2-PF0-OSC_IN)
- C9 pad 2: Net-(U2-(TIM4_CH3/TIM16_CH1/GPIO_EXTI8)PB8-BOOT0) -> Net-(U2-PF1-OSC_OUT)
- F3 pad 1: +12V -> /+12VIN
- F3 pad 2: Net-(F3-Pad2) -> +12V
- J1 pad 1: Net-(F3-Pad2) -> /+12VIN
- U2 pad 10: /SHDN.EMETER -> /SHDN.TSMP
- U2 pad 11: /SHDN.HVD -> /SHDN.MPC
- U2 pad 12: /SHDN.BSPD -> /SHDN.BMS
- U2 pad 13: /SHDN.BOTS -> /SHDN.HVD
- U2 pad 18: /SHDN.IS -> /SHDN.BSPD
- U2 pad 19: /SHDN.AIR-N -> /SHDN.BOTS
- U2 pad 2: /HEARTBEAT -> Net-(U2-PF0-OSC_IN)
- U2 pad 20: /ESTOP.RIGHT -> /SHDN.IS
- U2 pad 25: /ESTOP.LEFT -> /HEARTBEAT
- U2 pad 26: /ESTOP.DRIVER -> /Debug1
- U2 pad 27: /Debug3 -> /Debug2
- U2 pad 28: /Debug2 -> /Debug3
- U2 pad 29: /Debug1 -> /ESTOP.DRIVER
- U2 pad 3: /SHDN.AIR-P -> Net-(U2-PF1-OSC_OUT)
- U2 pad 30: Net-(U2-(TIM3_CH4/TIM4_CH2/TIM17_CH1N/GPIO_EXTI7)PB7) -> /ESTOP.LEFT
- U2 pad 31: Net-(U2-(TIM4_CH3/TIM16_CH1/GPIO_EXTI8)PB8-BOOT0) -> /ESTOP.RIGHT
- U2 pad 5: /SHDN.TSMS -> /SHDN.IMD
- U2 pad 6: /SHDN.IMD -> /SHDN.TSMS
- U2 pad 7: /SHDN.BMS -> /SHDN.AIR-P
- U2 pad 8: /SHDN.MPC -> /SHDN.AIR-N
- U2 pad 9: /SHDN.TSMP -> /SHDN.EMETER
- U7 pad 5: +5V -> +3V3
- Y1 pad 1: Net-(U2-(TIM4_CH3/TIM16_CH1/GPIO_EXTI8)PB8-BOOT0) -> Net-(U2-PF1-OSC_OUT)
- Y1 pad 3: Net-(U2-(TIM3_CH4/TIM4_CH2/TIM17_CH1N/GPIO_EXTI7)PB7) -> Net-(U2-PF0-OSC_IN)
Routing:
- net +3V3: track 30.0 -> 1.74 mm
- net /SWDIO: track 13.5 -> 35.1 mm, vias 1 -> 0
- net GND: track 15.3 -> 34.8 mm, vias 50 -> 39
- net /SHDN.BOTS: track 22.0 -> 40.5 mm, vias 0 -> 2
- net /SHDN.IS: track 14.4 -> 31.8 mm
- net /SHDN.BSPD: track 37.0 -> 53.4 mm, vias 0 -> 2
- net /CAN_RX: track 21.3 -> 6.16 mm
- net /CAN_TX: track 17.9 -> 8.91 mm
- net Net-(U2-(TIM3_CH4/TIM4_CH2/TIM17_CH1N/GPIO_EXTI7)PB7): track 8.86 -> 0.00 mm
- net Net-(U2-(TIM4_CH3/TIM16_CH1/GPIO_EXTI8)PB8-BOOT0): track 8.69 -> 0.00 mm
- net Net-(U2-PF1-OSC_OUT): track 0.00 -> 8.45 mm
- net Net-(U2-PF0-OSC_IN): track 0.00 -> 8.11 mm
- net /SHDN.TSMP: track 27.9 -> 35.8 mm
- net /ESTOP.LEFT: track 53.3 -> 45.8 mm, vias 2 -> 0
- net /+12VIN: track 0.00 -> 7.43 mm
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Other:
- board text added: "C8"
- board text added: "CLK"
- board text added: "DIO"
- board text added: "HB"
- board text removed: "HEARTBEAT"
- board text removed: "NRST"
- board text removed: "SWDIO"

Commit message: final tweeks
Parts:
- added REF**: OEM_Logo_8mm, OEM:OEM_Logo_8mm, B.Cu at (259.4, 79.2)
- added kibuzzard-6A3E9A3A: G***, kibuzzard-6A3E9A3A, B.Cu at (251.1, 82.1)
- added kibuzzard-6A3E9A3F: G***, kibuzzard-6A3E9A3F, B.Cu at (248.4, 76.4)
- added kibuzzard-6A3E9B69: G***, kibuzzard-6A3E9B69, B.Cu at (247.1, 79.3)
