File: vehicle/mkviii/hardware/integration/continuity_test/single_board_method/LCD Display/continuity_test.kicad_sch (KiCad schematic)
At the start: 33 parts, among them J1 Conn_01x02_Pin, J2 Programming_Pin_Header, J3 Conn_01x02_Pin, U1 STM32G441KBT6, U2 MCP2561-E_SN, U3 AP63203WU-7, U4 TLV70450DBVR, Y1 X_Crystal_16MHz_18pF

Commit message: versions 1 2 and 3 added to repo
Parts:
- added U5: ER_OLEDM0.91_1x-I2C, Display:ER_OLEDM0.91_1x-I2C, symbol Display_Graphic:ER_OLEDM0.91_1x-I2C
Connections:
- net GND: now also U5.1 (GND)
- net SWCLK: no longer U1.24 ((SYS_JTCK-SWCLK/GPIO_EXTI14)PA14)
- net SWDIO: no longer U1.23 ((SYS_JTMS-SWDIO/GPIO_EXTI13)PA13)
- net ID0_debug: no longer names the net of U1.18 ((TIM4_ETR/USART1_CK/GPIO_EXTI8)PA8)
- net ID1_debug: no longer names the net of U1.19 ((TIM2_CH3/TIM15_BKIN/USART1_TX/GPIO_EXTI9)PA9)
- net ID2_debug: no longer names the net of U1.20 ((TIM2_CH4/USART1_RX/TIM17_BKIN/GPIO_EXTI10)PA10)
- net ID3_debug: no longer names the net of U1.25 ((TIM2_ETR/TIM2_CH1/GPIO_EXTI15)PA15)
- net ID4_debug: no longer names the net of U1.26 ((TIM3_ETR/SPI1_SCK/TIM4_ETR/TIM2_CH2/GPIO_EXTI3)PB3)
- net ID5_debug: no longer names the net of U1.27 ((TIM17_BKIN/SPI1_MISO/TIM3_CH1/TIM16_CH1/GPIO_EXTI4)PB4)
- net ID6_debug: no longer names the net of U1.28 ((TIM17_CH1/SPI1_MOSI/TIM3_CH2/TIM16_BKIN/GPIO_EXTI5)PB5)
- net ID7_debug: no longer names the net of U1.29 ((TIM4_CH1/TIM16_CH1N/GPIO_EXTI6)PB6)
- new net 3V3: U5.2 (VCC)
- new net I2C_SCL: U1.23 ((SYS_JTMS-SWDIO/GPIO_EXTI13)PA13), U5.3 (SCL)
- new net I2C_SDA: U1.24 ((SYS_JTCK-SWCLK/GPIO_EXTI14)PA14), U5.4 (SDA)
- no-connect marks 12 -> 20
Other:
- note added: "Board connects to CAN and powers LV line through external battery connected to back of board. STM32 listens over CAN for signals from each LV component that is connected to CAN and screen prints out list of boards it cant see or first one in list of boards it cannot see (as that is likely the origin of the issue)"
- note added: "LQFP32"
- note removed: "Board connects to CAN and powers LV line through external battery connected to back of board. STM32 listens over CAN for signals from each LV component that is connected to CAN and light for that component turns green when it has recieved at least 1 message from that board."

Commit message: split into 3 versions, screen variant pcb layout beginning
Parts:
- C1, C11, C12, C13, C14, C15, C2, C3, C4, C5, C6, C7, C8: footprint OEM:C_0603 -> OEM:C_0603_1608Metric
- C10, C18, C9: footprint Capacitor_SMD:C_1206_3216Metric -> OEM:C_0603_1608Metric
- D1, D2: footprint OEM:CHIPLED_0805 -> OEM:D_0805_2012Metric
- F1, F2, F3: footprint OEM:Fuse_1210 -> OEM:Fuse_1210_3225Metric
- J1, J3: footprint Connector:CUI_PD-30S -> Connector:Banana_Jack_2Pin
- J2: footprint stm32g441kbt6:Programming_Pin_Header_Keyed -> OEM:J_Programming_Pin_Header_Keyed
- L1: footprint stm32g441kbt6:IND_BOURNS_SRR5018 -> OEM:IND_BOURNS_SRR5018 (L_3.9uH_2A_55m_SMD)
- R1, R2, R3: footprint OEM:R_0603 -> OEM:R_0603_1608Metric
- U1: footprint stm32g441kbt6:STM32G441KBT6 -> OEM:LQFP-32_7x7mm_P0.8mm
- U2: footprint stm32g441kbt6:SOIC127P600X175-8N -> OEM:U_1.222V-Buck-Conv_RT6285GSP_ SOP-8
- U3: footprint stm32g441kbt6:AP63203WU-7_DIO -> OEM:SOT-23-6
- Y1: footprint OEM:Crystal_TXC7M -> OEM:FA238160000MBC0 (X_16MHz_18pF_SMD - FA-238_16.0000MB-C0)
Changed lines of the file:
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@@
 			)
 		)
-		(property "Footprint" "OEM:CHIPLED_0805"
+		(property "Footprint" "OEM:D_0805_2012Metric"
 			(at 222.25 25.4 0)
 			(hide yes)
@@
 			)
 		)
-		(property "Footprint" "OEM:R_0603"
+		(property "Footprint" "OEM:R_0603_1608Metric"
 			(at 257.81 27.178 90)
 			(hide yes)
@@
 			)
 		)
-		(property "Footprint" "Connector:CUI_PD-30S"
+		(property "Footprint" "Connector:Banana_Jack_2Pin"
 			(at 20.32 78.74 0)
 			(hide yes)
@@
 			)
 		)
-		(property "Footprint" "OEM:C_0603"
+		(property "Footprint" "OEM:C_0603_1608Metric"
 			(at 35.2552 147.32 0)
 			(hide yes)
@@
 			)
 		)
-		(property "Footprint" "OEM:C_0603"
+		(property "Footprint" "OEM:C_0603_1608Metric"
 			(at 236.22 99.3648 0)
 			(hide yes)
@@
 			)
 		)
-		(property "Footprint" "OEM:Fuse_1210"
+		(property "Footprint" "OEM:Fuse_1210_3225Metric"
 			(at 273.05 105.918 90)
 			(hide yes)
@@
 			)
 		)
-		(property "Footprint" "stm32g441kbt6:AP63203WU-7_DIO"
+		(property "Footprint" "OEM:SOT-23-6"
 			(at 215.9 104.14 0)
 			(hide yes)
@@
 			)
 		)
-		(property "Footprint" "OEM:R_0603"
+		(property "Footprint" "OEM:R_0603_1608Metric"
 			(at 210.82 27.178 90)
 			(hide yes)
@@
 			)
 		)
-		(property "Footprint" "Capacitor_SMD:C_1206_3216Metric"
+		(property "Footprint" "OEM:C_0603_1608Metric"
 			(at 263.8552 66.04 0)
 			(hide yes)
@@
 			)
 		)
-		(property "Footprint" "OEM:C_0603"
+		(property "Footprint" "OEM:C_0603_1608Metric"
 			(at 148.2852 120.65 0)
 			(hide yes)
@@
 			)
 		)
-		(property "Footprint" "OEM:C_0603"
+		(property "Footprint" "OEM:C_0603_1608Metric"
 			(at 18.7452 36.83 0)
 			(hide yes)
@@
 			)
 		)
-		(property "Footprint" "OEM:C_0603"
+		(property "Footprint" "OEM:C_0603_1608Metric"
 			(at 166.0652 140.97 0)
 			(hide yes)
@@
 			)
 		)
-		(property "Footprint" "OEM:CHIPLED_0805"
+		(property "Footprint" "OEM:D_0805_2012Metric"
 			(at 269.24 25.4 0)
 			(hide yes)
@@
 			)
 		)
-		(property "Footprint" "OEM:C_0603"
+		(property "Footprint" "OEM:C_0603_1608Metric"
 			(at 192.7352 115.57 0)
 			(hide yes)
@@
 			)
 		)
-		(property "Footprint" "OEM:C_0603"
+		(property "Footprint" "OEM:C_0603_1608Metric"
 			(at 20.0152 147.32 0)
 			(hide yes)
@@
 			)
 		)
-		(property "Footprint" "OEM:Fuse_1210"
+		(property "Footprint" "OEM:Fuse_1210_3225Metric"
 			(at 22.86 29.718 90)
 			(hide yes)
@@
 			)
 		)
-		(property "Footprint" "OEM:C_0603"
+		(property "Footprint" "OEM:C_0603_1608Metric"
 			(at 201.6252 67.31 0)
 			(hide yes)
@@
 			)
 		)
-		(property "Footprint" "stm32g441kbt6:SOIC127P600X175-8N"
+		(property "Footprint" "OEM:U_1.222V-Buck-Conv_RT6285GSP_ SOP-8"
 			(at 247.65 240.97 0)
 			(hide yes)
@@
 			)
 		)
-		(property "Footprint" "OEM:C_0603"
+		(property "Footprint" "OEM:C_0603_1608Metric"
 			(at 36.5252 120.65 0)
 			(hide yes)
@@
 			)
 		)
-		(property "Footprint" "OEM:R_0603"
+		(property "Footprint" "OEM:R_0603_1608Metric"
 			(at 247.142 146.05 90)
 			(hide yes)
@@
 			)
 		)
-		(property "Footprint" "OEM:Fuse_1210"
+		(property "Footprint" "OEM:Fuse_1210_3225Metric"
 			(at 269.24 58.928 90)
 			(hide yes)
@@
 			)
 		)
-		(property "Footprint" "OEM:C_0603"
+		(property "Footprint" "OEM:C_0603_1608Metric"
 			(at 184.4548 148.59 0)
 			(hide yes)
@@
 			)
 		)
-		(property "Footprint" "OEM:C_0603"
+		(property "Footprint" "OEM:C_0603_1608Metric"
 			(at 176.2252 127 0)
 			(hide yes)
@@
 			)
 		)
-		(property "Footprint" "stm32g441kbt6:STM32G441KBT6"
+		(property "Footprint" "OEM:LQFP-32_7x7mm_P0.8mm"
 			(at 99.06 152.4 0)
 			(hide yes)
@@
 			)
 		)
-		(property "Footprint" "OEM:Crystal_TXC7M"
+		(property "Footprint" "OEM:FA238160000MBC0 (X_16MHz_18pF_SMD - FA-238_16.0000MB-C0)"
 			(at 170.18 118.11 0)
 			(hide yes)
@@
 			)
 		)
-		(property "Footprint" "Capacitor_SMD:C_1206_3216Metric"
+		(property "Footprint" "OEM:C_0603_1608Metric"
 			(at 253.6952 113.03 0)
 			(hide yes)
@@
 			)
 		)
-		(property "Footprint" "stm32g441kbt6:Programming_Pin_Header_Keyed"
+		(property "Footprint" "OEM:J_Programming_Pin_Header_Keyed"
 			(at 35.56 175.26 0)
 			(hide yes)
@@
 			)
 		)
-		(property "Footprint" "Capacitor_SMD:C_1206_3216Metric"
+		(property "Footprint" "OEM:C_0603_1608Metric"
 			(at 267.6652 113.03 0)
 			(hide yes)
@@
 			)
 		)
-		(property "Footprint" "OEM:C_0603"
+		(property "Footprint" "OEM:C_0603_1608Metric"
 			(at 20.0152 120.65 0)
 			(hide yes)
@@
 			)
 		)
-		(property "Footprint" "OEM:C_0603"
+		(property "Footprint" "OEM:C_0603_1608Metric"
 			(at 53.0352 120.65 0)
 			(hide yes)
@@
 			)
 		)
-		(property "Footprint" "Connector:CUI_PD-30S"
+		(property "Footprint" "Connector:Banana_Jack_2Pin"
 			(at 20.32 57.15 0)
 			(hide yes)
@@
 			)
 		)
-		(property "Footprint" "stm32g441kbt6:IND_BOURNS_SRR5018"
+		(property "Footprint" "OEM:IND_BOURNS_SRR5018 (L_3.9uH_2A_55m_SMD)"
 			(at 243.84 104.14 0)
 			(hide yes)

Commit message: PCB design
Parts:
- added J4: Conn_01x02_Pin, Connector_Molex:Molex_Micro-Fit_3.0_43045-0412_2x02_P3.00mm_Vertical, symbol Connector:Conn_01x02_Pin
- added R4, R5: R_2.2k_0.1W, OEM:R_0603_1608Metric, symbol OEM:R_2.2k_0.1W_0603
- C10, C18, C9: footprint OEM:C_0603_1608Metric -> OEM:C_1206_3216Metric
- J1, J3: footprint Connector:Banana_Jack_2Pin -> Connector_Molex:Molex_Micro-Fit_3.0_43045-0412_2x02_P3.00mm_Vertical
Connections:
- net 3V3 is gone; now on net +3V3: U5.2 (VCC)
- net SWCLK is gone; now on net I2C_SDA: J2.5 (Pin_5)
- net SWDIO is gone; now on net I2C_SCL: J2.1 (Pin_1)
- net +12V: now also C12.1, F1.1, F1.2
- net +5V: no longer C12.1, F1.1
- net CAN_+: now also J4.1 (Pin_1)
- net CAN_-: now also J4.2 (Pin_2)
- net I2C_SCL: now also R4.1; no longer U5.3 (SCL)
- net I2C_SDA: now also R5.1; no longer U5.4 (SDA)
- new net: R4.2, U5.3 (SCL)
- new net: R5.2, U5.4 (SDA)
Other:
- moved on the sheet: U5
