File: vehicle/mkviii/hardware/hv/HV motherboard/air-ctrl.kicad_sch (KiCad schematic)
At the start: 1 part, among them J501 pcie_x1_air_ctrl

Commit message: didn't change anything but wtv.
Connections:
- net GND: now also J501.A3 (GND)
- net +3.3V: now reaches J501.A2 (12V/3V(DA_ONLY))
- no-connect marks 13 -> 11
Changed lines of the file:
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@@
-	)
-	(no_connect
-		(at 123.19 76.2)
 	)
 	(no_connect
@@
 		(at 123.19 114.3)
 	)
-	(no_connect
-		(at 123.19 83.82)
-	)
 	(wire
 		(pts
@@
 	(wire
 		(pts
-			(xy 115.57 78.74) (xy 123.19 78.74)
+			(xy 111.76 78.74) (xy 123.19 78.74)
 		)
 		(stroke
@@
 	(wire
 		(pts
-			(xy 115.57 77.47) (xy 115.57 78.74)
+			(xy 111.76 76.2) (xy 111.76 78.74)
 		)
 		(stroke
@@
 	(wire
 		(pts
+			(xy 118.11 76.2) (xy 123.19 76.2)
+		)
+		(stroke
+			(width 0)
+			(type default)
+		)
+	)
+	(wire
+		(pts
 			(xy 166.37 99.06) (xy 166.37 93.98)
 		)
@@
 			(width 0)
 			(type default)
+		)
+	)
+	(label "GND"
+		(at 123.19 83.82 180)
+		(effects
+			(font
+				(size 1.27 1.27)
+			)
+			(justify right bottom)
 		)
 	)
@@
 	(symbol
 		(lib_id "power:+5V")
-		(at 115.57 77.47 0)
+		(at 111.76 76.2 0)
 		(unit 1)
 		(body_style 1)
@@
 		(dnp no)
 		(property "Reference" "#PWR?"
-			(at 115.57 81.28 0)
+			(at 111.76 80.01 0)
 			(hide yes)
 			(show_name no)
@@
 		)
 		(property "Value" "+5V"
-			(at 115.57 72.39 0)
+			(at 111.76 71.12 0)
 			(show_name no)
 			(do_not_autoplace no)
@@
 		)
 		(property "Footprint" ""
-			(at 115.57 77.47 0)
+			(at 111.76 76.2 0)
 			(hide yes)
 			(show_name no)
@@
 		)
 		(property "Datasheet" ""
-			(at 115.57 77.47 0)
+			(at 111.76 76.2 0)
 			(hide yes)
 			(show_name no)
@@
 		)
 		(property "Description" ""
-			(at 115.57 77.47 0)
-			(hide yes)
-			(show_name no)
+			(at 111.76 76.2 0)
+			(hide yes)
+			(show_name no)
+			(do_not_autoplace no)
+			(effects
+				(font
+					(size 1.27 1.27)
+				)
+			)
+		)
+		(pin "1"
+		)
+		(instances
+			(project "motherboard-pcie"
+				(path "/8f26d479-2c33-489f-a4df-6bb31c904ceb/59e3884a-39d0-4f6c-bd8f-e4f897fa95a0"
+					(reference "#PWR?")
+					(unit 1)
+				)
+			)
+		)
+	)
+	(symbol
+		(lib_id "power:+3.3V")
+		(at 118.11 76.2 0)
+		(unit 1)
+		(body_style 1)
+		(exclude_from_sim no)
+		(in_bom yes)
+		(on_board yes)
+		(in_pos_files yes)
+		(dnp no)
+		(fields_autoplaced yes)
+		(property "Reference" "#PWR?"
+			(at 118.11 80.01 0)
+			(hide yes)
+			(show_name no)
+			(do_not_autoplace no)
+			(effects
+				(font
+					(size 1.27 1.27)
+				)
+			)
+		)
+		(property "Value" "+3.3V"
+			(at 118.11 71.12 0)
+			(show_name no)
+			(do_not_autoplace no)
+			(effects
+				(font
+					(size 1.27 1.27)
+				)
+			)
+		)
+		(property "Footprint" ""
+			(at 118.11 76.2 0)
+			(hide yes)
+			(show_name no)
+			(do_not_autoplace no)
+			(effects
+				(font
+					(size 1.27 1.27)
+				)
+			)
+		)
+		(property "Datasheet" ""
+			(at 118.11 76.2 0)
+			(hide yes)
+			(show_name no)
+			(do_not_autoplace no)
+			(effects
+				(font
+					(size 1.27 1.27)
+				)
+			)
+		)
+		(property "Description" "Power symbol creates a global label with name \"+3.3V\""
+			(at 118.11 76.2 0)
+			(hide yes)
+			(show_name no)
