File: vehicle/mkviii/hardware/hv/HV motherboard/bms-core.kicad_sch (KiCad schematic)
At the start: 1 part, among them J801 pcie_x1_bms_core

Commit message: didn't change anything but wtv.
Parts:
- removed J801: pcie_x1_bms_core, OEM:te_pcie_x1_connector, symbol OEM:pcie_x1
- added J5: J_PCIe_x1, OEM:J_PCIe_x1_Key, symbol OEM:J_PCIe_x1
Connections:
- net +5V: now also J5.B5 (5V)
- net BSPD_CURRENT_THRESH: now also J5.B7 (io_3)
- net CAN+: now also J5.A4 (CAN+)
- net CAN-: now also J5.A5 (CAN-)
- net FAN_PWM: now also J5.B6 (io_1)
- net GND: now also J5.A3 (GND), J5.A6 (io_0), J5.A7 (io_2), J5.A8 (io_4), J5.A9 (io_6), J5.B4 (GND)
- net SHDN_SENSE_BMS: now also J5.B17 (SHDN_OUT/io_23), J5.B18 (SHDN_OUT/io_25)
- net SHDN_SENSE_MPC: now also J5.A17 (SHDN_IN/io_22), J5.A18 (SHDN_IN/io_24)
- net VOUT_CURRENT_SENSE: now also J5.B8 (io_5)
- new net 3.3V: J5.A2 (3.3V)
- no-connect marks 20 -> 19
Changed lines of the file:
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@@
-	)
-	(no_connect
-		(at 124.46 76.2)
 	)
 	(no_connect
@@
 		(pts
 			(xy 124.46 121.92) (xy 124.46 123.19)
+		)
+		(stroke
+			(width 0)
+			(type default)
+		)
+	)
+	(wire
+		(pts
+			(xy 120.65 76.2) (xy 124.46 76.2)
 		)
 		(stroke
@@
 			)
 		)
-		(property "Value" "+5V"
+		(property "Value" "3.3V"
 			(at 116.84 73.66 0)
 			(show_name no)
@@
 				(path "/8f26d479-2c33-489f-a4df-6bb31c904ceb/32c032b6-d9da-4a02-a2b0-a101292be82a"
 					(reference "#PWR?")
+					(unit 1)
+				)
+			)
+		)
+	)
+	(symbol
+		(lib_id "OEM:J_PCIe_x1")
+		(at 142.24 97.79 0)
+		(unit 1)
+		(body_style 1)
+		(exclude_from_sim no)
+		(in_bom yes)
+		(on_board yes)
+		(in_pos_files yes)
+		(dnp no)
+		(fields_autoplaced yes)
+		(property "Reference" "J5"
+			(at 142.24 67.31 0)
+			(show_name no)
+			(do_not_autoplace yes)
+			(effects
+				(font
+					(size 1.27 1.27)
+				)
+			)
+		)
+		(property "Value" "J_PCIe_x1"
+			(at 142.24 69.85 0)
+			(show_name no)
+			(do_not_autoplace yes)
+			(effects
+				(font
+					(size 1.27 1.27)
+				)
+			)
+		)
+		(property "Footprint" "OEM:J_PCIe_x1_Key"
+			(at 142.24 62.23 0)
+			(hide yes)
+			(show_name no)
+			(do_not_autoplace no)
+			(effects
+				(font
+					(size 1.27 1.27)
+				)
+			)
+		)
+		(property "Datasheet" "https://www.te.com/commerce/DocumentDelivery/DDEController?Action=showdoc&DocId=Data+Sheet%7F4-1773442-7%7F0308%7Fpdf%7FEnglish%7FENG_DS_4-1773442-7_0308.pdf%7F2-1761465-1"
+			(at 143.51 64.77 0)
+			(hide yes)
+			(show_name no)
+			(do_not_autoplace no)
+			(effects
+				(font
+					(size 1.27 1.27)
+				)
+			)
+		)
+		(property "Description" "Interface used to connect daugterboards to motherboards"
+			(at 142.24 97.79 0)
+			(hide yes)
+			(show_name no)
+			(do_not_autoplace no)
+			(effects
+				(font
+					(size 1.27 1.27)
+				)
+			)
+		)
+		(property "MPN" "2-1761465-1"
+			(at 142.24 97.79 0)
+			(hide yes)
+			(show_name no)
+			(do_not_autoplace no)
+			(effects
+				(font
+					(size 1.27 1.27)
+				)
+			)
+		)
+		(pin "A18"
+		)
+		(pin "B18"
+		)
+		(pin "B4"
+		)
+		(pin "A7"
+		)
+		(pin "A8"
+		)
+		(pin "A9"
+		)
+		(pin "B6"
+		)
+		(pin "A2"
+		)
+		(pin "A10"
+		)
+		(pin "B7"
+		)
+		(pin "A15"
+		)
+		(pin "B14"
+		)
+		(pin "A13"
+		)
+		(pin "A6"
+		)
+		(pin "A12"
+		)
+		(pin "A4"
+		)
+		(pin "B11"
+		)
+		(pin "B12"
+		)
+		(pin "A17"
+		)
+		(pin "B15"
+		)
+		(pin "A5"
+		)
+		(pin "A14"
+		)
+		(pin "B10"
+		)
+		(pin "B8"
+		)
+		(pin "B13"
+		)
+		(pin "A16"
+		)
+		(pin "A11"
+		)
+		(pin "B2"
+		)
+		(pin "B9"
+		)
+		(pin "B16"
+		)
+		(pin "A3"
+		)
+		(pin "B17"
+		)
+		(pin "B3"
+		)
+		(pin "A1"
+		)
+		(pin "B1"
+		)
+		(pin "B5"
+		)
+		(instances
+			(project "motherboard-pcie"
+				(path "/8f26d479-2c33-489f-a4df-6bb31c904ceb/32c032b6-d9da-4a02-a2b0-a101292be82a"
+					(reference "J5")
 					(unit 1)
 				)
@@
 	)
 	(symbol
-		(lib_id "OEM:pcie_x1")
-		(at 142.24 97.79 0)
+		(lib_name "+5V_1")
+		(lib_id "power:+5V")
+		(at 120.65 76.2 0)
 		(unit 1)
 		(body_style 1)
@@
 		(in_pos_files yes)
 		(dnp no)
-		(property "Reference" "J801"
-			(at 142.24 67.31 0)
-			(show_name no)
-			(do_not_autoplace yes)
-			(effects
-				(font
-					(size 1.27 1.27)
-				)
-			)
-		)
-		(property "Value" "pcie_x1_bms_core"
-			(at 142.24 69.85 0)
-			(show_name no)
-			(do_not_autoplace yes)
-			(effects
-				(font
-					(size 1.27 1.27)
-				)
-			)
-		)
-		(property "Footprint" "OEM:te_pcie_x1_connector"
-			(at 142.24 62.23 0)
-			(hide yes)
-			(show_name no)
-			(do_not_autoplace no)
-			(effects
-				(font
-					(size 1.27 1.27)
-				)
-			)
-		)
-		(property "Datasheet" "https://www.te.com/commerce/DocumentDelivery/DDEController?Action=showdoc&DocId=Data+Sheet%7F4-1773442-7%7F0308%7Fpdf%7FEnglish%7FENG_DS_4-1773442-7_0308.pdf%7F2-1761465-1"
-			(at 143.51 64.77 0)
-			(hide yes)
-			(show_name no)
-			(do_not_autoplace no)
-			(effects
-				(font
-					(size 1.27 1.27)
-				)
-			)
-		)
-		(property "Description" ""
-			(at 142.24 97.79 0)
-			(hide yes)
-			(show_name no)
-			(do_not_autoplace no)
-			(effects
-				(font
-					(size 1.27 1.27)
-				)
-			)
-		)
-		(pin "B16"
-		)
-		(pin "A4"
-		)
-		(pin "A5"
-		)
-		(pin "A6"
-		)
-		(pin "B8"
-		)
-		(pin "B6"
-		)
-		(pin "B17"
-		)
-		(pin "B3"
-		)
-		(pin "A18"
-		)
-		(pin "A3"
-		)
-		(pin "B12"
-		)
-		(pin "A17"
-		)
-		(pin "A7"
-		)
-		(pin "A2"
-		)
-		(pin "B4"
-		)
-		(pin "A16"
-		)
-		(pin "B13"
-		)
-		(pin "B11"
-		)
-		(pin "B10"
-		)
-		(pin "A9"
-		)
-		(pin "B7"
-		)
-		(pin "B2"
-		)
-		(pin "B18"
-		)
-		(pin "B9"
-		)
-		(pin "B5"
-		)
-		(pin "B15"
-		)
-		(pin "A10"
-		)
-		(pin "A8"
-		)
-		(pin "B1"
-		)
-		(pin "A1"
-		)
-		(pin "A13"
-		)
-		(pin "A14"
-		)
-		(pin "A12"
-		)
-		(pin "A11"
-		)
-		(pin "A15"
-		)
-		(pin "B14"
+		(fields_autoplaced yes)
+		(property "Reference" "#PWR?"
+			(at 120.65 80.01 0)
+			(hide yes)
+			(show_name no)
+			(do_not_autoplace no)
+			(effects
+				(font
+					(size 1.27 1.27)
+				)
+			)
+		)
+		(property "Value" "+5V"
+			(at 120.65 71.12 0)
+			(show_name no)
+			(do_not_autoplace no)
+			(effects
+				(font
+					(size 1.27 1.27)
+				)
+			)
+		)
+		(property "Footprint" ""
+			(at 120.65 76.2 0)
+			(hide yes)
+			(show_name no)
+			(do_not_autoplace no)
+			(effects
+				(font
+					(size 1.27 1.27)
+				)
+			)
+		)
+		(property "Datasheet" ""
+			(at 120.65 76.2 0)
+			(hide yes)
+			(show_name no)
+			(do_not_autoplace no)
+			(effects
+				(font
+					(size 1.27 1.27)
+				)
+			)
+		)
+		(property "Description" "Power symbol creates a global label with name \"+5V\""
+			(at 120.65 76.2 0)
+			(hide yes)
+			(show_name no)
+			(do_not_autoplace no)
+			(effects
+				(font
+					(size 1.27 1.27)
+				)
+			)
+		)
+		(pin "1"
 		)
 		(instances
 			(project "motherboard-pcie"
 				(path "/8f26d479-2c33-489f-a4df-6bb31c904ceb/32c032b6-d9da-4a02-a2b0-a101292be82a"
-					(reference "J801")
+					(reference "#PWR?")
 					(unit 1)
 				)
