File: vehicle/mkviii/hardware/integration/pdu_sg/shdn_in_conversion.kicad_sch (KiCad schematic)
At the start: 15 parts, among them Q1 SSM3K333R, Q2 SSM3K333R, Q3 SSM3K333R

Commit message: fix symbols after changing library
Parts:
- D31, D32, D33: footprint OEM:D_0805_2012Metric -> Diode_SMD:D_0805_2012Metric
- Q1, Q2, Q3: footprint OEM:SOT-23-3 -> Package_TO_SOT_SMD:SOT-23-3
- R37, R38, R39, R40, R41, R42, R43, R44, R46: footprint OEM:R_0603_1608Metric -> Resistor_SMD:R_0603_1608Metric
Changed lines of the file:
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@@
 			)
 		)
-		(property "Footprint" "OEM:R_0603_1608Metric"
+		(property "Footprint" "Resistor_SMD:R_0603_1608Metric"
 			(at 248.412 111.76 90)
 			(hide yes)
@@
 			)
 		)
-		(property "Footprint" "OEM:R_0603_1608Metric"
+		(property "Footprint" "Resistor_SMD:R_0603_1608Metric"
 			(at 169.672 111.76 90)
 			(hide yes)
@@
 			)
 		)
-		(property "Footprint" "OEM:SOT-23-3"
+		(property "Footprint" "Package_TO_SOT_SMD:SOT-23-3"
 			(at 144.78 104.14 0)
 			(hide yes)
@@
 			)
 		)
-		(property "Footprint" "OEM:D_0805_2012Metric"
+		(property "Footprint" "Diode_SMD:D_0805_2012Metric"
 			(at 80.01 116.84 0)
 			(hide yes)
@@
 			)
 		)
-		(property "Footprint" "OEM:R_0603_1608Metric"
+		(property "Footprint" "Resistor_SMD:R_0603_1608Metric"
 			(at 158.242 111.76 90)
 			(hide yes)
@@
 			)
 		)
-		(property "Footprint" "OEM:R_0603_1608Metric"
+		(property "Footprint" "Resistor_SMD:R_0603_1608Metric"
 			(at 71.882 111.76 90)
 			(hide yes)
@@
 			)
 		)
-		(property "Footprint" "OEM:R_0603_1608Metric"
+		(property "Footprint" "Resistor_SMD:R_0603_1608Metric"
 			(at 83.312 111.76 90)
 			(hide yes)
@@
 			)
 		)
-		(property "Footprint" "OEM:R_0603_1608Metric"
+		(property "Footprint" "Resistor_SMD:R_0603_1608Metric"
 			(at 236.982 111.76 90)
 			(hide yes)
@@
 			)
 		)
-		(property "Footprint" "OEM:SOT-23-3"
+		(property "Footprint" "Package_TO_SOT_SMD:SOT-23-3"
 			(at 58.42 104.14 0)
 			(hide yes)
@@
 			)
 		)
-		(property "Footprint" "OEM:R_0603_1608Metric"
+		(property "Footprint" "Resistor_SMD:R_0603_1608Metric"
 			(at 59.182 95.25 90)
 			(hide yes)
@@
 			)
 		)
-		(property "Footprint" "OEM:D_0805_2012Metric"
+		(property "Footprint" "Diode_SMD:D_0805_2012Metric"
 			(at 245.11 116.84 0)
 			(hide yes)
@@
 			)
 		)
-		(property "Footprint" "OEM:R_0603_1608Metric"
+		(property "Footprint" "Resistor_SMD:R_0603_1608Metric"
 			(at 224.282 95.25 90)
 			(hide yes)
@@
 			)
 		)
-		(property "Footprint" "OEM:D_0805_2012Metric"
+		(property "Footprint" "Diode_SMD:D_0805_2012Metric"
 			(at 166.37 116.84 0)
 			(hide yes)
@@
 			)
 		)
-		(property "Footprint" "OEM:SOT-23-3"
+		(property "Footprint" "Package_TO_SOT_SMD:SOT-23-3"
 			(at 223.52 104.14 0)
 			(hide yes)
@@
 			)
 		)
-		(property "Footprint" "OEM:R_0603_1608Metric"
+		(property "Footprint" "Resistor_SMD:R_0603_1608Metric"
 			(at 145.542 95.25 90)
 			(hide yes)
