File: vehicle/mkviii/hardware/integration/pdu_sg/buck_can.kicad_sch (KiCad schematic)
At the start: 4 parts, among them U9 TLV70450DBVR

Commit message: 5v regulator for can
Parts:
- removed C16: C_0.1uF_16V, OEM:C_0603_1608Metric, symbol OEM:C_0.1uF_16V_0603
- added C16: C_0.47uF, OEM:C_0603_1608Metric, symbol OEM:C_0.47uF_25V_0603
- added D11: Green_LED, OEM:D_0805_2012Metric, symbol OEM:D_LED_Green_0805
- added D12: D_Red_LED, OEM:D_0805_2012Metric, symbol OEM:D_LED_Red_0805
- added R10: R_499, OEM:R_0603_1608Metric, symbol OEM:R_499_0.1W_0603
- added R11: R_200_0.1W, OEM:R_0603_1608Metric, symbol OEM:R_200_0.1W_0603
- added TP4: TP_SMD, OEM:TP_Hook_SMD, symbol OEM_mkvii:TP_Hook_SMD
- C17: value C_0.1uF_16V -> C_0.1uF
Connections:
- net 5V_buck_vin: now also R10.1
- net 5V_buck_vout: now also C16.1, R11.1, TP4.1
- net GND: now also C16.2, D11.1 (K), D12.1 (K)
- new net: D11.2 (A), R10.2
- new net: D12.2 (A), R11.2
- no-connect marks 0 -> 2

Commit message: 5v buck convertor for can
Other:
- note added: "12V to 5V Buck Convertor"
- moved on the sheet: C16, C17, D10, D11, D12, R10, R11, TP4, U9

Commit message: lv power distribution + rs232
Parts:
- D12: value D_Red_LED -> Red_LED
- R11: value R_200_0.1W -> R_200
Changed lines of the file:
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@@
 			)
 		)
-		(property "Value" "R_200_0.1W"
+		(property "Value" "R_200"
 			(at 191.77 114.2999 0)
 			(show_name no)
@@
 			)
 		)
-		(property "Value" "D_Red_LED"
+		(property "Value" "Red_LED"
 			(at 193.04 123.5074 90)
 			(show_name no)

Commit message: fix symbols after changing library
Parts:
- D11, D12: footprint OEM:D_0805_2012Metric -> Diode_SMD:D_0805_2012Metric
- R10, R11: footprint OEM:R_0603_1608Metric -> Resistor_SMD:R_0603_1608Metric
- U9: footprint OEM:SOT-23-5 -> Package_TO_SOT_SMD:SOT-23-5
Changed lines of the file:
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@@
 			)
 		)
-		(property "Footprint" "OEM:R_0603_1608Metric"
+		(property "Footprint" "Resistor_SMD:R_0603_1608Metric"
 			(at 103.632 107.95 90)
 			(hide yes)
@@
 			)
 		)
-		(property "Footprint" "OEM:R_0603_1608Metric"
+		(property "Footprint" "Resistor_SMD:R_0603_1608Metric"
 			(at 187.452 113.03 90)
 			(hide yes)
@@
 			)
 		)
-		(property "Footprint" "OEM:SOT-23-5"
+		(property "Footprint" "Package_TO_SOT_SMD:SOT-23-5"
 			(at 160.02 192.71 0)
 			(hide yes)
@@
 			)
 		)
-		(property "Footprint" "OEM:D_0805_2012Metric"
+		(property "Footprint" "Diode_SMD:D_0805_2012Metric"
 			(at 189.23 120.65 0)
 			(hide yes)
@@
 			)
 		)
-		(property "Footprint" "OEM:D_0805_2012Metric"
+		(property "Footprint" "Diode_SMD:D_0805_2012Metric"
 			(at 105.41 118.11 0)
 			(hide yes)

Commit message: fix footprints
Parts:
- C16, C17: footprint OEM:C_0603_1608Metric -> Capacitor_SMD:C_0603_1608Metric
Changed lines of the file:
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@@
 			)
 		)
-		(property "Footprint" "OEM:C_0603_1608Metric"
+		(property "Footprint" "Capacitor_SMD:C_0603_1608Metric"
 			(at 127.9652 111.76 0)
 			(hide yes)
@@
 			)
 		)
-		(property "Footprint" "OEM:C_0603_1608Metric"
+		(property "Footprint" "Capacitor_SMD:C_0603_1608Metric"
 			(at 171.1452 116.84 0)
 			(hide yes)
