File: vehicle/mkviii/hardware/lv/wheel_speed/wheel_speed_Testing_Things.kicad_sch (KiCad schematic)
At the start: 35 parts, among them J1 J_Programming_Pin_Header, J2 pcie_x1, Q1 SSM3K333R, Q2 SSM3K333R, U1 STM32G441KBT6, U2 MCP2561-E-SN, Y1 Crystal_16MHz_18pF

Commit message: DR2
Parts:
- removed D1, D2: LED_BLUE, OEM:CHIPLED_0805, symbol OEM:LED_BLUE
- removed R4, R9: R_100, OEM:R_0603, symbol OEM:R
- added D3, D4: D_Blue_LED, Diode_SMD:D_0805_2012Metric, symbol OEM:D_LED_Blue_0805
- added R1, R3: R_60.4, Resistor_SMD:R_0603_1608Metric, symbol OEM:R_60.4_0.1W_0603
Connections:
- net +3V3: now also J2.A2 (12V/3V(DA_ONLY)); no longer C3.2, J2.B5 (5V), U2.3 (VDD)
- net DEBUG_LED: now also D3.2 (A)
- net GND: now also R1.2, R3.2
- net HEARTBEAT_LED: now also D4.2 (A)
- new net: D3.1 (K), R1.1
- new net: D4.1 (K), R3.1
- new net +5: C3.2, U2.3 (VDD)
- new net +5V: J2.B5 (5V)
- no-connect marks 45 -> 44

Commit message: DR2
Parts:
- removed C1, C3, C6: C_0.1uF, OEM:C_0603, symbol OEM:0u1F
- removed C2: C_10nF, OEM:C_0603, symbol OEM:0u1F
- removed C3: 0u1F, OEM:C_0603, symbol OEM:0u1F
- removed C4: C_1uF, OEM:C_0603, symbol OEM:0u1F
- removed C5: C_4.7uF, OEM:C_0603, symbol OEM:0u1F
- removed C6, C7: 10nF, OEM:C_0603, symbol OEM:C
- removed C7, C8: C_30pF, OEM:C_0603, symbol OEM:0u1F
- removed J2: pcie_x1, OEM:pcie_x1, symbol OEM:pcie_x1
- removed Q1, Q2: SSM3K333R, OEM:SOT-23F, symbol OEM:SSM3K333R
- removed R2: R_120_DNP, OEM:R_0603, symbol OEM:R
- removed R5, R7: 1K, OEM:R_0603, symbol OEM:R
- removed R6, R8: R_1K_DNP, OEM:R_0603, symbol OEM:R
- removed TP1, TP2: TP_SMD, OEM:Test_Point_SMD, symbol OEM:TP_SMD
- removed Y1: Crystal_16MHz_18pF, OEM:Crystal_TXC7M, symbol OEM:Crystal_16MHz_18pF
- added C1, C10, C11: C_10nF, Capacitor_SMD:C_0603_1608Metric, symbol OEM:C_10nF_20-100V_0603
- added C2, C3, C8: C_0.1uF, Capacitor_SMD:C_0603_1608Metric, symbol OEM:C_0.1uF_20-100V_0603
- added C4: C_1uF, Capacitor_SMD:C_0603_1608Metric, symbol OEM:C_1uF_20-100V_0603
- added C5: C_0.1uF, Capacitor_SMD:C_0603_1608Metric, symbol OEM:C_0.1uF_0-20V_0603
- added C6: C_4.7uF, Capacitor_SMD:C_0603_1608Metric, symbol OEM:C_4.7uF_20-100V_0603
- added C7, C9: C_30pF, Capacitor_SMD:C_0603_1608Metric, symbol OEM:C_30pF_20-100V_0603
- added Can_Testpoint1, Can_Testpoint2: TestPoint, TestPoint:TestPoint_Pad_D1.0mm, symbol OEM:TP_1mm
- added J2: J_PCIe_x1, OEM:J_PCIe_x1_Key, symbol OEM:J_PCIe_x1
- added Q1, Q2: SSM3K333R,LF, Package_TO_SOT_SMD:SOT-23-3, symbol OEM:Q_NMOS_30V_6A_SOT-23F
- added R1: R_120, Resistor_SMD:R_0603_1608Metric, symbol OEM:R_120_0.1W_0603
- added R4, R5, R7, R8: R_1k, Resistor_SMD:R_0603_1608Metric, symbol OEM:R_1k_0.1W_0603
- added X1: X_16MHz_18pF, OEM:FA238160000MBC0 (X_16MHz_18pF_SMD - FA-238_16.0000MB-C0), symbol OEM:X_16MHz_18pF_SMD
- renumbered D3 to D1, D4 to D2, R1 to R2, U2 to U1, U1 to U2, WS1_Input to WS1_Input1, WS1_Output to WS1_Output1, WS2_Input to WS2_Input1, WS2_Output to WS2_Output1
Connections:
- net +3V3: now also C1.1, C2.1, C3.1, C4.1, C6.1, J2.A2 (12V/3V(DA_ONLY)), R7.1, R8.1
- net +5: now also C5.2
- net +5V: now also J2.B5 (5V)
- net CAN_+: now also Can_Testpoint1.1, J2.A4 (CAN+), R1.1
- net CAN_-: now also Can_Testpoint2.1, J2.A5 (CAN-), R1.2
- net GND: now also C1.2, C10.2, C11.2, C2.2, C3.2, C4.2, C5.1, C6.2, C7.2, C8.2, C9.2, J2.A3 (GND), J2.B4 (GND), Q1.2 (S), Q2.2 (S), X1.2, X1.4
- net RESET: now also C8.1
- net ws1_Vout: now also J2.B8 (io_5), R4.1
- net ws1_fVout: now also Q1.3 (D), R8.2
- net ws2_Vout: now also J2.B6 (io_1), R5.1
- net ws2_fVout: now also Q2.3 (D), R7.2
- net at U2.2 ((EVENTOUT/TIM1_CH3N/SPI2_NSS/I2C2_WS/I2C2_SDA)PF0-OSC_IN): now also C9.1, X1.3
- net at U2.3 ((EVENTOUT/SPI2_SCK)PF1-OSC_OUT): now also C7.1, X1.1
- net at WS1_Input1.1: now also C10.1, Q1.1 (G), R4.2
- net at WS2_Input1.1: now also C11.1, Q2.1 (G), R5.2
Other:
- note removed: "X_16MHz_18pF"
