File: vehicle/mkviii/hardware/integration/PDU/PDU.kicad_pcb (KiCad board)
At the start: 2 copper layers, 182 parts, among them J1 J_PCIe_x1, J10 CONN_02x03, J11 CONN_02x03, J12 CONN_01X03, J13 CONN_01X03, J14 CONN_01X03, J2 CONN_DSub-9, J3 J_PCIe_x1, J4 J_PCIe_x1, J5 CONN_02x03, J6 CONN_01X03, J7 J_Programming_Pin_Header, J8 CONN_01X03, J9 CONN_02x03, K1 G5Q-1A4-DC5, Q1 SSM3K333R, Q10 SSM3K333R, Q2 SSM3K333R, Q3 SSM3K333R, Q6 SSM3K333R, Q7 SSM3K333R, Q8 SSM3K333R, Q9 SSM3K333R, U1 STM32G441KBT6, U2 MCP23S17_SS, U20 ADC1283, U21 MAX7221xNG, U3 TLV70450DBVR, U4 CC56-12SEKWA, U5 AP63203WU-7, U6 MCP2561-E_SN, Y1 X_Crystal_16MHz_18pF

Commit message: Sort the parts together
Parts:
- moved D18 244.7 mm to (442.9, 196.0), turned to 180 degrees
- moved D19 242.0 mm to (442.9, 191.5), turned to 180 degrees
- moved D20 239.4 mm to (442.9, 187.0), turned to 180 degrees
- moved C11 238.1 mm to (433.5, 182.2), turned to -90 degrees
- moved R31 237.4 mm to (438.5, 187.0)
- moved C3 237.3 mm to (98.5, 133.6)
- moved C5 237.3 mm to (98.5, 138.6)
- moved D21 237.2 mm to (442.9, 183.0), turned to 180 degrees
- moved D33 237.1 mm to (442.9, 200.5), turned to 180 degrees
- moved U4 236.9 mm to (385.8, -33.5)
- moved R5 236.9 mm to (74.0, 148.8), turned to -90 degrees
- moved U21 235.6 mm to (410.9, -39.0)
- moved R44 235.5 mm to (438.5, 196.0)
- moved R47 235.3 mm to (438.5, 200.5)
- moved D22 235.1 mm to (442.9, 178.5), turned to 180 degrees
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Connections:
- D15 pad 1: /CAN_5+ -> /CAN_5-
- D15 pad 2: /CAN_5- -> /CAN_5+
- D31 pad 1: GND -> /INVERTER_FAULT
- D32 pad 1: GND -> /INVERTER_START_OK
- R17 pad 1: /INVERTER_START_OK -> +5V
- R5 pad 1: /INVERTER_FAULT -> +5V
Other:
- board text added: "5V buck"
- board text added: "8-segment Display"
- board text added: "ADC"
- board text added: "CAN"
- board text added: "Cooling out"
- board text added: "Fan PWM"
- board text added: "Low Voltage Power Distribution"
- board text added: "Pump PWM"
- board text added: "STM32"
- board text added: "Shutdown circuits"
- board text added: "Status LEDs"
- board text added: "TS Stat"
